File: devboard/esp32-c1_devboard.rev2/esp32-c1_devboard.sch (KiCad schematic (older format))
At the start: 41 parts, among them J1 USB_C, J2 Conn_02x10_Odd_Even, J3 Conn_02x10_Odd_Even, Q1 S8050, Q2 S8050, SW1 SW_SPST, SW2 SW_SPST, U1 ESP32-C3-MINI-1, U2 CH340C, U4 AP1117-33

Commit message: rev
Parts:
- gave numbers to parts that had none: 4
Changed lines of the file:
@@
 $EndComp
 $Comp
-L Device:LED D?
+L Device:LED D1
 U 1 1 61CD9E0D
 P 6300 5900
-F 0 "D?" V 6339 5782 50  0000 R CNN
+F 0 "D1" V 6339 5782 50  0000 R CNN
 F 1 "LED" V 6248 5782 50  0000 R CNN
 F 2 "LED_SMD:LED_0805_2012Metric" H 6300 5900 50  0001 C CNN
@@
 $EndComp
 $Comp
-L Device:R R?
+L Device:R R12
 U 1 1 61CDC4AD
 P 6300 6250
-F 0 "R?" H 6370 6296 50  0000 L CNN
+F 0 "R12" H 6370 6296 50  0000 L CNN
 F 1 "10K" H 6370 6205 50  0000 L CNN
 F 2 "Resistor_SMD:R_0402_1005Metric" V 6230 6250 50  0001 C CNN
@@
 $EndComp
 $Comp
-L power:GND #PWR?
+L power:GND #PWR0124
 U 1 1 61CDD051
 P 6300 6450
-F 0 "#PWR?" H 6300 6200 50  0001 C CNN
+F 0 "#PWR0124" H 6300 6200 50  0001 C CNN
 F 1 "GND" H 6305 6277 50  0000 C CNN
 F 2 "" H 6300 6450 50  0001 C CNN
@@
 $EndComp
 $Comp
-L Device:LED D?
+L Device:LED D2
 U 1 1 61CDD69C
 P 6950 4950
-F 0 "D?" H 6943 4695 50  0000 C CNN
+F 0 "D2" H 6943 4695 50  0000 C CNN
 F 1 "LED" H 6943 4786 50  0000 C CNN
 F 2 "LED_SMD:LED_0805_2012Metric" H 6950 4950 50  0001 C CNN
@@
 $EndComp
 $Comp
-L Device:R R?
+L Device:R R14
 U 1 1 61CDDACF
 P 7300 4950
-F 0 "R?" H 7370 4996 50  0000 L CNN
+F 0 "R14" H 7370 4996 50  0000 L CNN
 F 1 "10K" H 7370 4905 50  0000 L CNN
 F 2 "Resistor_SMD:R_0402_1005Metric" V 7230 4950 50  0001 C CNN
@@
 $EndComp
 $Comp
-L power:GND #PWR?
+L power:GND #PWR0125
 U 1 1 61CDE177
 P 7500 5000
-F 0 "#PWR?" H 7500 4750 50  0001 C CNN
+F 0 "#PWR0125" H 7500 4750 50  0001 C CNN
 F 1 "GND" H 7505 4827 50  0000 C CNN
 F 2 "" H 7500 5000 50  0001 C CNN
